File: board/board.kicad_pcb (KiCad board)
At the start: 2 copper layers, 21 x 13 mm, 1 part

Commit message: initial
Parts:
- added D1: MB2S, Package_TO_SOT_SMD:TO-269AA, F.Cu at (150.6, 93.5)
- added D2: MB2S, Package_TO_SOT_SMD:TO-269AA, F.Cu at (150.6, 99.3)
- added J1: 004_BASE-T_CT, on_edge:on_edge_2x05_device, F.Cu at (140.0, 96.5)
- added J2: 013_PoE_rectified, on_edge:on_edge_2x05_host, F.Cu at (161.0, 96.5)
- LOGO1: moved to B.Cu
- turned LOGO1 to 180 degrees
Routing:
- net Net-(J1-Pad1): track 0.00 -> 28.3 mm, vias 0 -> 3
- net GND: track 0.00 -> 21.4 mm, vias 0 -> 2
- net /rectifier/CT3: track 0.00 -> 17.3 mm, vias 0 -> 1
- net /rectifier/48V: track 0.00 -> 17.1 mm
- net /rectifier/CT2: track 0.00 -> 13.4 mm
- net /rectifier/CT4: track 0.00 -> 5.56 mm, vias 0 -> 1
- net /rectifier/CT1: track 0.00 -> 5.29 mm
Other:
- outline, holes or cut-outs redrawn
