File: board/board.kicad_sch (KiCad schematic)
At the start: 1 part

Commit message: initial
Parts:
- added J1: 004_BASE-T_CT, on_edge:on_edge_2x05_device, symbol put_on_edge:004_BASE-T_CT
- added J2: 013_PoE_rectified, on_edge:on_edge_2x05_host, symbol put_on_edge:013_PoE_rectified
Connections:
- new net: J1.1 (GND), J1.10 (GND), J1.3 (GND), J1.5 (GND), J1.7 (GND), J1.9 (GND)
- new net GND: J2.1 (GND), J2.2 (GND), J2.5 (GND)
- new net rectifier/48V: J2.3 (48V), J2.4 (48V)
- new net rectifier/CT1: J1.2 (CT1)
- new net rectifier/CT2: J1.4 (CT2)
- new net rectifier/CT3: J1.6 (CT3)
- new net rectifier/CT4: J1.8 (CT4)
Other:
- sheet implementation renamed rectifier
- sheet rectifier: file implementation.kicad_sch -> rectifier.kicad_sch
- sheet rectifier ports: added 48V, CT1, CT2, CT3, CT4, GND; removed none
- note removed: "Input connectors go here"
- note removed: "Output connectors go here"
Changed lines of the file:
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@@
 (kicad_sch (version 20211123) (generator eeschema)
   (paper "A4")
-  (text "Output connectors go here" (at 224.79 88.9 0)
-    (effects (font (size 1.27 1.27)) (justify left bottom))
-  )
-  (text "Input connectors go here" (at 49.53 88.9 0)
-    (effects (font (size 1.27 1.27)) (justify left bottom))
+  (junction (at 187.96 105.41) (diameter 0) (color 0 0 0 0)
+  )
+  (junction (at 203.2 125.73) (diameter 0) (color 0 0 0 0)
+  )
+  (junction (at 88.9 123.19) (diameter 0) (color 0 0 0 0)
+  )
+  (junction (at 91.44 123.19) (diameter 0) (color 0 0 0 0)
+  )
+  (junction (at 93.98 123.19) (diameter 0) (color 0 0 0 0)
+  )
+  (junction (at 200.66 125.73) (diameter 0) (color 0 0 0 0)
+  )
+  (junction (at 86.36 123.19) (diameter 0) (color 0 0 0 0)
+  )
+  (wire (pts (xy 93.98 123.19) (xy 96.52 123.19))
+    (stroke (width 0) (type default) (color 0 0 0 0))
+  )
+  (wire (pts (xy 101.6 105.41) (xy 114.3 105.41))
+    (stroke (width 0) (type default) (color 0 0 0 0))
+  )
+  (wire (pts (xy 88.9 120.65) (xy 88.9 123.19))
+    (stroke (width 0) (type default) (color 0 0 0 0))
+  )
+  (wire (pts (xy 101.6 110.49) (xy 114.3 110.49))
+    (stroke (width 0) (type default) (color 0 0 0 0))
+  )
+  (wire (pts (xy 203.2 125.73) (xy 203.2 127))
+    (stroke (width 0) (type default) (color 0 0 0 0))
+  )
+  (wire (pts (xy 175.26 125.73) (xy 200.66 125.73))
+    (stroke (width 0) (type default) (color 0 0 0 0))
+  )
+  (wire (pts (xy 200.66 125.73) (xy 203.2 125.73))
+    (stroke (width 0) (type default) (color 0 0 0 0))
+  )
+  (wire (pts (xy 205.74 124.46) (xy 205.74 125.73))
+    (stroke (width 0) (type default) (color 0 0 0 0))
+  )
+  (wire (pts (xy 91.44 123.19) (xy 93.98 123.19))
+    (stroke (width 0) (type default) (color 0 0 0 0))
+  )
+  (wire (pts (xy 93.98 120.65) (xy 93.98 123.19))
+    (stroke (width 0) (type default) (color 0 0 0 0))
+  )
+  (wire (pts (xy 187.96 107.95) (xy 187.96 105.41))
+    (stroke (width 0) (type default) (color 0 0 0 0))
+  )
+  (wire (pts (xy 205.74 125.73) (xy 203.2 125.73))
+    (stroke (width 0) (type default) (color 0 0 0 0))
+  )
+  (wire (pts (xy 200.66 124.46) (xy 200.66 125.73))
+    (stroke (width 0) (type default) (color 0 0 0 0))
+  )
+  (wire (pts (xy 86.36 120.65) (xy 86.36 123.19))
+    (stroke (width 0) (type default) (color 0 0 0 0))
+  )
+  (wire (pts (xy 175.26 105.41) (xy 187.96 105.41))
+    (stroke (width 0) (type default) (color 0 0 0 0))
+  )
+  (wire (pts (xy 101.6 102.87) (xy 114.3 102.87))
+    (stroke (width 0) (type default) (color 0 0 0 0))
+  )
+  (wire (pts (xy 86.36 123.19) (xy 88.9 123.19))
+    (stroke (width 0) (type default) (color 0 0 0 0))
+  )
+  (wire (pts (xy 187.96 105.41) (xy 190.5 105.41))
+    (stroke (width 0) (type default) (color 0 0 0 0))
+  )
+  (wire (pts (xy 101.6 107.95) (xy 114.3 107.95))
+    (stroke (width 0) (type default) (color 0 0 0 0))
+  )
+  (wire (pts (xy 96.52 123.19) (xy 96.52 120.65))
+    (stroke (width 0) (type default) (color 0 0 0 0))
+  )
+  (wire (pts (xy 190.5 107.95) (xy 187.96 107.95))
+    (stroke (width 0) (type default) (color 0 0 0 0))
+  )
+  (wire (pts (xy 91.44 120.65) (xy 91.44 123.19))
+    (stroke (width 0) (type default) (color 0 0 0 0))
+  )
+  (wire (pts (xy 88.9 123.19) (xy 91.44 123.19))
+    (stroke (width 0) (type default) (color 0 0 0 0))
+  )
+  (wire (pts (xy 83.82 120.65) (xy 83.82 123.19))
+    (stroke (width 0) (type default) (color 0 0 0 0))
+  )
+  (wire (pts (xy 83.82 123.19) (xy 86.36 123.19))
+    (stroke (width 0) (type default) (color 0 0 0 0))
+  )
+  (wire (pts (xy 203.2 125.73) (xy 203.2 124.46))
+    (stroke (width 0) (type default) (color 0 0 0 0))
+  )
+  (symbol (lib_id "put_on_edge:004_BASE-T_CT") (at 90.17 106.68 0) (mirror y) (unit 1)
+    (in_bom yes) (on_board yes) (fields_autoplaced)
+    (property "Reference" "J1" (id 0) (at 90.805 88.9 0))
+    (property "Value" "004_BASE-T_CT" (id 1) (at 90.805 91.44 0))
+    (property "Footprint" "on_edge:on_edge_2x05_device" (id 2) (at 82.55 90.17 0)
+      (effects (font (size 1.27 1.27)) hide)
+    )
+    (property "Datasheet" "" (id 3) (at 82.55 90.17 0)
+      (effects (font (size 1.27 1.27)) hide)
+    )
+    (pin "1")
+    (pin "10")
+    (pin "2")
+    (pin "3")
+    (pin "4")
+    (pin "5")
+    (pin "6")
+    (pin "7")
+    (pin "8")
+    (pin "9")
+  )
+  (symbol (lib_id "power:GND") (at 203.2 127 0) (unit 1)
+    (in_bom yes) (on_board yes) (fields_autoplaced)
+    (property "Reference" "#PWR0101" (id 0) (at 203.2 133.35 0)
+      (effects (font (size 1.27 1.27)) hide)
+    )
+    (property "Value" "GND" (id 1) (at 203.2 132.08 0))
+    (property "Footprint" "" (id 2) (at 203.2 127 0)
+      (effects (font (size 1.27 1.27)) hide)
+    )
+    (property "Datasheet" "" (id 3) (at 203.2 127 0)
+      (effects (font (size 1.27 1.27)) hide)
+    )
+    (pin "1")
   )
   (symbol (lib_id "Graphic:Logo_Open_Hardware_Small") (at 273.05 157.48 0) (unit 1)
@@
       (effects (font (size 1.27 1.27)) hide)
     )
+  )
+  (symbol (lib_id "put_on_edge:013_PoE_rectified") (at 201.93 110.49 0) (unit 1)
+    (in_bom yes) (on_board yes) (fields_autoplaced)
+    (property "Reference" "J2" (id 0) (at 210.82 108.5849 0)
+      (effects (font (size 1.27 1.27)) (justify left))
+    )
+    (property "Value" "013_PoE_rectified" (id 1) (at 210.82 111.1249 0)
+      (effects (font (size 1.27 1.27)) (justify left))
+    )
+    (property "Footprint" "on_edge:on_edge_2x05_host" (id 2) (at 209.55 93.98 0)
+      (effects (font (size 1.27 1.27)) hide)
+    )
+    (property "Datasheet" "" (id 3) (at 209.55 93.98 0)
+      (effects (font (size 1.27 1.27)) hide)
+    )
+    (pin "1")
+    (pin "2")
+    (pin "3")
+    (pin "4")
+    (pin "5")
   )
   (sheet (at 114.3 72.39) (size 60.96 62.23) (fields_autoplaced)
     (stroke (width 0.1524) (type solid) (color 0 0 0 0))
     (fill (color 0 0 0 0.0000))
-    (property "Sheet name" "implementation" (id 0) (at 114.3 71.6784 0)
+    (property "Sheet name" "rectifier" (id 0) (at 114.3 71.6784 0)
       (effects (font (size 1.27 1.27)) (justify left bottom))
     )
-    (property "Sheet file" "implementation.kicad_sch" (id 1) (at 114.3 135.2046 0)
+    (property "Sheet file" "rectifier.kicad_sch" (id 1) (at 114.3 135.2046 0)
       (effects (font (size 1.27 1.27)) (justify left top))
+    )
+    (pin "GND" input (at 175.26 125.73 0)
+      (effects (font (size 1.27 1.27)) (justify right))
+    )
+    (pin "48V" input (at 175.26 105.41 0)
+      (effects (font (size 1.27 1.27)) (justify right))
+    )
+    (pin "CT1" input (at 114.3 102.87 180)
+      (effects (font (size 1.27 1.27)) (justify left))
+    )
+    (pin "CT2" input (at 114.3 105.41 180)
+      (effects (font (size 1.27 1.27)) (justify left))
+    )
+    (pin "CT3" input (at 114.3 107.95 180)
+      (effects (font (size 1.27 1.27)) (justify left))
+    )
+    (pin "CT4" input (at 114.3 110.49 180)
+      (effects (font (size 1.27 1.27)) (justify left))
     )
   )
@@
   )
   (symbol_instances
+    (path "/2e943e4c-3252-4ad1-a735-fa97e130638d"
+      (reference "#PWR0101") (unit 1) (value "GND") (footprint "")
+    )
+    (path "/767ce4c6-0e55-4543-92f0-34cb8237a544/7f5f8093-49f9-4dd2-8910-45ffcd8f5757"
+      (reference "D1") (unit 1) (value "MB2S") (footprint "Package_TO_SOT_SMD:TO-269AA")
+    )
+    (path "/767ce4c6-0e55-4543-92f0-34cb8237a544/e04157dc-c0fa-446a-9352-86efb8cefc27"
+      (reference "D2") (unit 1) (value "MB2S") (footprint "Package_TO_SOT_SMD:TO-269AA")
+    )
+    (path "/2a1e6d18-c0c2-40e2-8486-875a0f7aa380"
+      (reference "J1") (unit 1) (value "004_BASE-T_CT") (footprint "on_edge:on_edge_2x05_device")
+    )
+    (path "/ff3484d9-b44b-4f1b-8abc-9854280ab743"
+      (reference "J2") (unit 1) (value "013_PoE_rectified") (footprint "on_edge:on_edge_2x05_host")
+    )
     (path "/b72b6f4a-7489-40f2-bb90-d75ae01aa368"
       (reference "LOGO1") (unit 1) (value "Logo_Open_Hardware_Small") (footprint "Symbol:OSHW-Symbol_6.7x6mm_SilkScreen")
